File: line_follower.kicad_pcb (KiCad board)
At the start: 2 copper layers, 151.1 x 176.3 mm, 108 parts, among them J1 Conn_01x20_Socket, J10 Conn_01x20_Pin, J11 Conn_01x20_Pin, J12 Conn_01x02_Socket, J13 Conn_01x04_Pin, J2 Conn_01x20_Socket, J3 Conn_01x06_Socket, J4 Conn_01x06_Socket, J5 XT60-M, J6 Conn_01x02_Socket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

Commit message: new schematic complete
Parts:
- removed 1, 2, 3, 4: MountingHole_2.1mm, MountingHole:MountingHole_2.1mm
- added 10: MountingHole_2.1mm, MountingHole:MountingHole_2.1mm, F.Cu at (143.6, 143.0)
- added 9: MountingHole_2.1mm, MountingHole:MountingHole_2.1mm, F.Cu at (128.6, 142.9)
- added REF**: N20 Motor Without Encoder, ROBO misc footprints:N20 Motor Without Encoder, F.Cu at (70.1, 194.8)
- added REF**: N20 Motor Mount, ROBO misc footprints:N20 Motor Mount, F.Cu at (70.1, 194.8)
- added REF**: N20 Motor Mount, ROBO misc footprints:N20 Motor Mount, F.Cu at (204.4, 194.1)
- added REF**: N20 Motor Without Encoder, ROBO misc footprints:N20 Motor Without Encoder, F.Cu at (204.4, 194.1)
- C22, C23: footprint Capacitor_SMD:C_0603_1608Metric_Pad1.08x0.95mm_HandSolder -> Capacitor_Tantalum_SMD:CP_EIA-3528-12_Kemet-T_HandSolder
- moved R34 1.87 mm to (148.3, 232.2)
- moved C22 1.02 mm to (87.6, 185.1)
- moved G*** 0.88 mm to (135.9, 112.4)
- moved C23 0.76 mm to (101.4, 188.1)
Routing:
- net GND: track 148.8 -> 127.7 mm
- net /CALIB: track 90.6 -> 93.1 mm
- net /5V_STM: track 420.3 -> 418.9 mm
- net /3.3V_LDO: track 427.9 -> 427.1 mm
Other:
- outline, holes or cut-outs redrawn
- board text added: "BOT KILL"
- board text added: "DRV IN"
- board text added: "DRV OUT"
- board text added: "EN"
- board text added: "GND"
- board text added: "IN"
- board text added: "MOTOR KILL"
- board text added: "OUT"
- board text added: "PRIORITY"
- board text added: "RX"
- board text added: "STATE"
- board text added: "STM USB side"
- board text added: "TX"
- board text added: "VCC"
- board text removed: "MOTOR MOUNTS"
