File: line_follower.kicad_sch (KiCad schematic)
At the start: 97 parts, among them J1 Conn_01x20_Socket, J10 Conn_01x20_Pin, J11 Conn_01x20_Pin, J12 Conn_01x02_Socket, J13 Conn_01x04_Pin, J2 Conn_01x20_Socket, J3 Conn_01x06_Socket, J4 Conn_01x06_Socket, J5 XT60-M, J6 Conn_01x02_Socket, J7 Conn_01x02_Socket, J8 Conn_01x06_Socket, J9 Conn_01x02_Socket, SW1 SW_Push_DPDT, SW3 SW_Push_DPDT, SW4 SW_Push_DPDT, SW5 SW_Push, U1 AMS1117-3.3

Commit message: final pcb
Parts:
- added R33, R34: 10k, Resistor_SMD:R_0603_1608Metric_Pad0.98x0.95mm_HandSolder, symbol Device:R
Connections:
- net 3.3V_STM_1: now also SW5.1
- net CALIB: now also R34.2
- net GND: now also R33.2, R34.1; no longer SW5.1
- net PB9: now also R33.1
Changed lines of the file:
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@@
 		(color 0 0 0 0)
 	)
+	(junction
+		(at 31.75 111.76)
+		(diameter 0)
+		(color 0 0 0 0)
+	)
 	(no_connect
 		(at 303.53 44.45)
@@
 	(wire
 		(pts
+			(xy 252.73 46.99) (xy 252.73 50.8)
+		)
+		(stroke
+			(width 0)
+			(type default)
+		)
+	)
+	(wire
+		(pts
 			(xy 71.12 44.45) (xy 59.69 44.45)
 		)
@@
 	(wire
 		(pts
+			(xy 259.08 46.99) (xy 252.73 46.99)
+		)
+		(stroke
+			(width 0)
+			(type default)
+		)
+	)
+	(wire
+		(pts
 			(xy 105.41 82.55) (xy 105.41 85.09)
 		)
@@
 	(wire
 		(pts
-			(xy 31.75 107.95) (xy 31.75 111.76)
+			(xy 31.75 104.14) (xy 31.75 111.76)
 		)
 		(stroke
@@
 	(wire
 		(pts
+			(xy 252.73 58.42) (xy 252.73 60.96)
+		)
+		(stroke
+			(width 0)
+			(type default)
+		)
+	)
+	(wire
+		(pts
 			(xy 59.69 34.29) (xy 62.23 34.29)
 		)
@@
 		)
 	)
+	(label "GND"
+		(at 39.37 111.76 0)
+		(effects
+			(font
+				(size 1.27 1.27)
+			)
+			(justify left bottom)
+		)
+	)
 	(label "BUCK_IN"
 		(at 92.71 74.93 180)
@@
 		)
 	)
+	(label "GND"
+		(at 252.73 60.96 0)
+		(effects
+			(font
+				(size 1.27 1.27)
+			)
+			(justify left bottom)
+		)
+	)
 	(label "BUCK_IN"
 		(at 303.53 39.37 0)
@@
 	)
 	(label "PRIORITY"
-		(at 31.75 107.95 0)
+		(at 31.75 104.14 0)
 		(effects
 			(font
@@
 		)
 	)
-	(label "GND"
+	(label "3.3V_STM_1"
 		(at 31.75 121.92 270)
 		(effects
@@
 	(symbol
 		(lib_id "Device:R")
+		(at 252.73 54.61 180)
+		(unit 1)
+		(exclude_from_sim no)
+		(in_bom yes)
+		(on_board yes)
+		(dnp no)
+		(property "Reference" "R34"
+			(at 250.444 54.356 90)
+			(effects
+				(font
+					(size 1.27 1.27)
+				)
+			)
+		)
+		(property "Value" "10k"
+			(at 252.73 54.61 90)
+			(effects
+				(font
+					(size 1.27 1.27)
+				)
+			)
+		)
+		(property "Footprint" "Resistor_SMD:R_0603_1608Metric_Pad0.98x0.95mm_HandSolder"
+			(at 254.508 54.61 90)
+			(effects
+				(font
+					(size 1.27 1.27)
+				)
+				(hide yes)
+			)
+		)
+		(property "Datasheet" "~"
+			(at 252.73 54.61 0)
+			(effects
+				(font
+					(size 1.27 1.27)
+				)
+				(hide yes)
+			)
+		)
+		(property "Description" "Resistor"
+			(at 252.73 54.61 0)
+			(effects
+				(font
+					(size 1.27 1.27)
+				)
+				(hide yes)
+			)
+		)
+		(pin "1"
+		)
+		(pin "2"
+		)
+		(instances
+			(project "line_follower"
+				(path "/33f398db-e9fd-40e3-b7af-8ed3645b8356"
+					(reference "R34")
+					(unit 1)
+				)
+			)
+		)
+	)
+	(symbol
+		(lib_id "Device:R")
 		(at 246.38 168.91 270)
 		(unit 1)
@@
 					(unit 1)
 				)
+			)
+		)
+	)
+	(symbol
+		(lib_id "Device:R")
+		(at 35.56 111.76 90)
+		(unit 1)
+		(exclude_from_sim no)
+		(in_bom yes)
+		(on_board yes)
+		(dnp no)
+		(property "Reference" "R33"
+			(at 35.56 109.728 90)
+			(effects
+				(font
+					(size 1.27 1.27)
+				)
+			)
+		)
+		(property "Value" "10k"
+			(at 35.306 111.76 90)
+			(effects
+				(font
+					(size 1.27 1.27)
+				)
+			)
+		)
+		(property "Footprint" "Resistor_SMD:R_0603_1608Metric_Pad0.98x0.95mm_HandSolder"
+			(at 35.56 113.538 90)
+			(effects
+				(font
+					(size 1.27 1.27)
+				)
+				(hide yes)
+			)
+		)
+		(property "Datasheet" "~"
+			(at 35.56 111.76 0)
+			(effects
+				(font
+					(size 1.27 1.27)
+				)
+				(hide yes)
+			)
+		)
+		(property "Description" "Resistor"
+			(at 35.56 111.76 0)
+			(effects
+				(font
+					(size 1.27 1.27)
+				)
+				(hide yes)
+			)
+		)
+		(pin "1"
+		)
+		(pin "2"
+		)
+		(instances
+			(project ""
+				(path "/33f398db-e9fd-40e3-b7af-8ed3645b8356"
+					(reference "R33")
+					(unit 1)
+				)

Commit message: new schematic complete
Parts:
- removed C13, C14, C15, C16, C17, C18, C19, C20, C21: 0.1u, Capacitor_SMD:C_0603_1608Metric_Pad1.08x0.95mm_HandSolder, symbol Device:C
- removed D10, D11, D12, D13, D14, D2, D3, D4, D5, D6, D7, D8, D9: LED, LED_SMD:LED_0805_2012Metric_Pad1.15x1.40mm_HandSolder, symbol Device:LED
- removed J12, J6, J7, J9: Conn_01x02_Socket, Connector_PinSocket_2.54mm:PinSocket_1x02_P2.54mm_Vertical, symbol Connector:Conn_01x02_Socket
- removed J13: Conn_01x04_Pin, Connector_PinHeader_2.54mm:PinHeader_1x04_P2.54mm_Vertical, symbol Connector:Conn_01x04_Pin
- removed J3, J4: Conn_01x06_Socket, Connector_PinSocket_2.54mm:PinSocket_1x06_P2.54mm_Vertical, symbol Connector:Conn_01x06_Socket
- removed R23, R24, R25, R26, R27, R28, R29, R30, R31, R32: 150, Resistor_SMD:R_0603_1608Metric_Pad0.98x0.95mm_HandSolder, symbol Device:R
- removed R33, R34: 10k, Resistor_SMD:R_0603_1608Metric_Pad0.98x0.95mm_HandSolder, symbol Device:R
- removed SW3: SW_Push_DPDT, Button_Switch_THT:SW_Push_2P2T_Toggle_CK_PVA2xxH3xxxxxxV2, symbol Switch:SW_Push_DPDT
- added B1: ~, symbol ROBO misc symbols:MP1584_Mini_Buck
- added D2: ~, symbol ROBO misc symbols:DRV8833
- added J3: Conn_01x04_Pin, symbol Connector:Conn_01x04_Pin
- added J4: Conn_01x04_Socket, symbol Connector:Conn_01x04_Socket
- added J6, J7: Conn_02x05_Counter_Clockwise, symbol Connector_Generic:Conn_02x05_Counter_Clockwise
- added SW2, SW3: SW_Push, symbol Switch:SW_Push
- C22, C23: footprint Capacitor_SMD:C_0603_1608Metric_Pad1.08x0.95mm_HandSolder -> Capacitor_Tantalum_SMD:CP_EIA-3528-12_Kemet-T_HandSolder
- R20, R21, R22: value 150 -> 10k; footprint Resistor_SMD:R_0603_1608Metric_Pad0.98x0.95mm_HandSolder -> (none)
- SW5: footprint Button_Switch_THT:SW_PUSH_6mm_H5mm -> (none)
Connections:
- net LEFT is gone; now on net PC13: J1.19 (Pin_19), J11.19 (Pin_19)
- net 3.3V_LDO: now also C10.1, C11.1, C12.1, C3.1, C5.1, C6.1, C7.1, C8.1, C9.1, R11.2, R12.2, R13.2, R14.2, R15.2, R16.2, R17.2, R18.2, R19.2; no longer A1.4, A2.4, A3.4, A4.4, A5.4, A6.4, A7.4, A8.4, A9.4
- net 5V_STM: now also D1.2 (A), B1.3 (OUT+), J4.3 (Pin_3), J6.1 (Pin_1), J7.1 (Pin_1); no longer R10.1, R2.1, R3.1, R4.1, R5.1, R6.1, R7.1, R8.1, R9.1
- net BUCK_IN: now also B1.2 (IN+); no longer D1.2 (A)
- net GND: now also A1.3, A2.3, A3.3, A4.3, A5.3, A6.3, A7.3, A8.3, A9.3, R20.2, R21.2, R22.2, B1.1 (IN-), B1.4 (OUT-), D2.10 (GND), J4.4 (Pin_4); no longer R11.1, R12.1, R13.1, R14.1, R15.1, R16.1, R17.1, R18.1, R19.1
- net PA1: now also A8.4, R19.1; no longer A1.3, R11.2
- net PA12: now also R6.1, J6.10 (Pin_10), J7.10 (Pin_10)
- net PA15: now also R5.1, J6.9 (Pin_9), J7.9 (Pin_9)
- net PA2: now also A7.4, R12.1; no longer A2.3, R12.2
- net PA3: now also A6.4, R13.1; no longer A3.3, R13.2
- net PA4: now also A5.4, R14.1; no longer A4.3, R14.2
- net PA5: now also A4.4, R15.1; no longer A5.3, R15.2
- net PA6: now also A3.4, R16.1; no longer A6.3, R16.2
- net PA7: now also A2.4, R17.1; no longer A7.3, R17.2
- net PB0: now also A1.4, R18.1; no longer A8.3, R18.2
- net PB1: now also J8.6 (Pin_6); no longer A9.3, R19.2
- net PB10: now also D2.1 (EEP)
- net PB12: now also R10.1, J6.2 (Pin_2), J7.2 (Pin_2); no longer R20.2
- net PB13: now also R9.1, J6.3 (Pin_3), J7.3 (Pin_3); no longer R21.2
- net PB14: now also R8.1, J6.4 (Pin_4), J7.4 (Pin_4); no longer R22.2
- net PB2: now also J8.1 (Pin_1)
- net PB3: now also R4.1, J6.8 (Pin_8), J7.8 (Pin_8)
- net PB4: now also R3.1, J6.7 (Pin_7), J7.7 (Pin_7)
- net PB5: now also R2.1, J6.6 (Pin_6), J7.6 (Pin_6); no longer J8.1 (Pin_1)
- net PB9: now also J4.1 (Pin_1); no longer SW5.2
- net PC14: now also R21.1, SW3.1
- net PC15: now also R20.1, SW2.1
- net RPR_ANO_1: now also A1.1, R10.2; no longer A9.1, C12.1, R2.2
- net RPR_ANO_2: now also A2.1, R9.2; no longer A8.1, C11.1, R3.2
- net RPR_ANO_3: now also A3.1, R8.2; no longer A7.1, C10.1, R4.2
- net RPR_ANO_4: now also A4.1, R7.2; no longer A6.1, C9.1, R5.2
- net RPR_ANO_5: no longer C8.1
- net RPR_ANO_6: now also A6.1, R5.2; no longer A4.1, C7.1, R7.2
- net RPR_ANO_7: now also A7.1, R4.2; no longer A3.1, C6.1, R8.2
- net RPR_ANO_8: now also A8.1, R3.2; no longer A2.1, C5.1, R9.2
- net RPR_ANO_9: now also A9.1, R2.2; no longer A1.1, C3.1, R10.2
- net VCC_DRV: now also D2.9 (Vcc)
- net PC13: now reaches R22.1
- net PC13: now also SW5.1
- net 3.3V_STM_1 renamed 3.3V_STM1
- net 3.3V_STM1: now also SW5.2, SW2.2, SW3.2; no longer SW5.1
- net CALIB renamed PA0
- net PA0: now also A9.4, R11.1
- net EEP renamed PB15
- net PB15: now also R7.1, J6.5 (Pin_5), J7.5 (Pin_5)
- net EN renamed PB8
- net PB8: now also J4.2 (Pin_2); no longer J8.6 (Pin_6)
- net IN1 renamed PA8
- net PA8: now also D2.7 (IN1)
- net IN2 renamed PA9
- net PA9: now also D2.8 (IN2)
- net IN3 renamed PA10
- net PA10: now also D2.11 (IN3)
- net IN4 renamed PA11
- net PA11: now also D2.12 (IN4)
- net VBAT_STM renamed VBAT
- new net: D2.2 (OUT1), J3.1 (Pin_1)
- new net: D2.3 (OUT2), J3.2 (Pin_2)
- new net: D2.4 (OUT3), J3.3 (Pin_3)
- new net: D2.5 (OUT4), J3.4 (Pin_4)
- no-connect marks 7 -> 5
Other:
- note added: "ANLG1"
- note added: "ANLG2"
- note added: "ANLG3"
- note added: "ANLG4"
- note added: "ANLG5"
- note added: "ANLG6"
- note added: "ANLG7"
- note added: "ANLG8"
- note added: "ANLG9"
- note added: "DOWN"
- note added: "EEP"
- note added: "EN"
- note added: "IR1"
- note added: "IR2"
- note added: "IR3"
- note added: "IR4"
- note added: "IR5"
- note added: "IR6"
- note added: "IR7"
- note added: "IR8"
- note added: "IR9"
- note added: "Kill only motor"
- note added: "Kill whole bot"
- note added: "Menu Navigation"
- note added: "OLED Display"
- note added: "Ribbon Jumper for IR leds"
- note added: "SELECT"
- note added: "STATE"
- note added: "STM32F411CEU6"
- note added: "TIM1CH1"
- note added: "TIM1CH2"
- note added: "TIM1CH3"
- note added: "TIM1CH4"
- note added: "UP"
- note removed: "CALIBRATION BUTTON"
- note removed: "For only motor"
- note removed: "For whole bot"
- note removed: "LEDS FOR CALIBRATION STATUS"
- note removed: "MISC Buttons"
- note removed: "PRIORITY SELECTION BUTTON AND LEDS"
- note removed: "STM32F411CUE6"
- moved on the sheet: A1, A2, A3, A4, A5, A6, A7, A8, A9, C1, C10, C11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
